File: EE/TestBoard1/TB1/TB1.kicad_pcb (KiCad board)
At the start: 2 copper layers, 33.5 x 76 mm, 45 parts, among them J1 Peg, J10 Peg, J11 Peg, J12 Peg, J13 Conn_01x02, J14 Peg, J15 Peg, J16 Peg, J17 Peg, J18 Peg, J19 Peg, J2 Peg, J20 Conn_01x03, J21 Conn_01x01, J3 Peg, J4 Peg, J5 Peg, J6 Peg, J7 Peg, J8 Peg, J9 Peg, U1 AH1381, U10 AH1381, U11 AH1381, U12 AH1381, U13 AH1381, U14 AH1381, U15 AH1381, U16 AH1381, U17 AH1381, U18 AH1381, U2 AH1381, U3 AH1381, U4 AH1381, U5 AH1381, U6 AH1381, U7 AH1381, U8 AH1381, U9 AH1381

Commit message: Finished TB1 for Magnet Test
Parts:
- moved J2 20.9 mm to (153.8, 105.5)
- moved J6 20.9 mm to (153.8, 115.5)
- moved U1 20.9 mm to (153.8, 101.5)
- moved U2 20.9 mm to (153.8, 119.5)
- moved J1 19.1 mm to (173.8, 105.6)
- moved J10 19.1 mm to (173.8, 115.6)
- moved U10 19.1 mm to (173.8, 119.6)
- moved U9 19.1 mm to (173.8, 101.6)
- moved J21 2.02 mm to (149.3, 110.3)
Routing:
- net VCC: track 0.00 -> 74.7 mm
- net /HO_2: track 59.4 -> 105.3 mm, vias 0 -> 8
- net /HO_1: track 59.4 -> 102.5 mm, vias 0 -> 10
- net /HO_0: track 59.0 -> 97.7 mm, vias 0 -> 8
- net VCCQ: track 8.06 -> 36.3 mm, vias 0 -> 2
- net /VCC1: track 31.3 -> 29.8 mm
- net /VCC2: track 27.2 -> 26.7 mm
Other:
- outline, holes or cut-outs redrawn
