File: EE/Main/MainBoard/Sensor_31_60.kicad_sch (KiCad schematic)
At the start: 3 parts

Commit message: Sensors attached to mainboard
Parts:
- removed J? (x3): Conn_02x13_Odd_Even, Connector_PinHeader_1.27mm:PinHeader_2x13_P1.27mm_Vertical, symbol Connector_Generic:Conn_02x13_Odd_Even
Connections:
- no-connect marks 6 -> 0
