File: EE/Main/MainBoard/Power.kicad_sch (KiCad schematic)
At the start: 14 parts

Commit message: Updated layout, and placement for main board
Parts:
- added P1: USB_C_Plug_USB2.0, Connector_USB:USB_C_Receptacle_GCT_USB4085, symbol Connector:USB_C_Plug_USB2.0
- C2, C3, C4, C5, C6: renamed from C?; footprint (none) -> Capacitor_SMD:C_0603_1608Metric
- R14, R15, R16: renamed from R?; footprint (none) -> Resistor_SMD:R_0402_1005Metric
- gave numbers to parts that had none: 6
Connections:
- net GND: now also P1.A1 (GND), P1.A12 (GND), P1.B1 (GND), P1.B12 (GND)
- net VBUS: now also P1.A4 (VBUS), P1.A9 (VBUS), P1.B4 (VBUS), P1.B9 (VBUS)
- no-connect marks 0 -> 5

Commit message: Routed PCB, Need SCL/SDA still
Parts:
- removed SW1: SW_SPST, symbol Switch:SW_SPST
- added R17, R18, R19, R20: 0, Resistor_SMD:R_0402_1005Metric, symbol Device:R
- added SW1: EG1206A, Library:EG1206A_EWI, symbol New_Library:EG1206A
- D1: footprint (none) -> LED_SMD:LED_0603_1608Metric
- J8: footprint (none) -> Connector_JST:JST_PH_B2B-PH-K_1x02_P2.00mm_Vertical
- L1: footprint (none) -> Inductor_SMD:L_0805_2012Metric; P/N (none) -> 74479775222A
Connections:
- net GND: now also R17.1, R18.1; no longer J8.2 (Pin_2)
- net VBAT: now also R19.2, R20.2, SW1.1; no longer J8.1 (Pin_1)
- net V_PRE_REG: now also SW1.2 (COM)
- new net: J8.2 (Pin_2), R18.2, R20.1
- new net: J8.1 (Pin_1), R17.2, R19.1
- no-connect marks 5 -> 8
Other:
- note added: "Battery Estimations: 5mA for MCU, 1mA for Power Good LED 6x2.5 for 7 segment. 1mA for Hall effects 4x2.5mA for Hall LEDs 10+1+15+5, ~=50mA"
- moved on the sheet: J8
Changed lines of the file:
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@@
   (junction (at 227.584 91.948) (diameter 0) (color 0 0 0 0)
   )
+  (junction (at 93.472 188.468) (diameter 0) (color 0 0 0 0)
+  )
   (junction (at 237.998 111.252) (diameter 0) (color 0 0 0 0)
   )
   (junction (at 238.76 111.252) (diameter 0) (color 0 0 0 0)
   )
+  (junction (at 93.472 185.928) (diameter 0) (color 0 0 0 0)
+  )
   (junction (at 256.54 92.71) (diameter 0) (color 0 0 0 0)
   )
+  (no_connect (at 158.242 116.84))
+  (no_connect (at 143.002 106.68))
+  (no_connect (at 163.322 106.68))
   (no_connect (at 140.462 68.072))
   (no_connect (at 163.322 47.752))
@@
     (effects (font (size 1.27 1.27)) (justify left bottom))
   )
+  (text "Battery Estimations:\n5mA for MCU, \n1mA for Power Good LED\n6x2.5 for 7 segment. \n1mA for Hall effects\n4x2.5mA for Hall LEDs\n10+1+15+5, ~=50mA"
+    (at 21.336 132.08 0)
+    (effects (font (size 1.27 1.27)) (justify left bottom))
+  )
   (text "Regulator" (at 226.06 22.606 0)
     (effects (font (size 1.27 1.27)) (justify left bottom))
@@
     (effects (font (size 1.27 1.27)) (justify left bottom))
   )
-  (label "V_PRE_REG" (at 143.256 94.742 0)
+  (label "V_PRE_REG" (at 153.162 102.87 0)
     (effects (font (size 1.27 1.27)) (justify left bottom))
   )
@@
     (effects (font (size 1.27 1.27)) (justify right bottom))
   )
-  (label "VBAT" (at 84.836 110.744 0)
-    (effects (font (size 1.27 1.27)) (justify left bottom))
-  )
-  (label "VBAT" (at 133.096 94.742 180)
+  (label "VBAT" (at 101.092 185.928 0)
+    (effects (font (size 1.27 1.27)) (justify left bottom))
+  )
+  (label "VBAT" (at 101.092 188.468 0)
+    (effects (font (size 1.27 1.27)) (justify left bottom))
+  )
+  (label "VBAT" (at 148.082 116.84 270)
     (effects (font (size 1.27 1.27)) (justify right bottom))
+  )
+  (symbol (lib_id "power:GND") (at 93.472 196.088 90) (unit 1)
+    (in_bom yes) (on_board yes) (fields_autoplaced)
+    (property "Reference" "#PWR0137" (id 0) (at 99.822 196.088 0)
+      (effects (font (size 1.27 1.27)) hide)
+    )
+    (property "Value" "GND" (id 1) (at 96.647 196.5218 90)
+      (effects (font (size 1.27 1.27)) (justify right))
+    )
+    (property "Footprint" "" (id 2) (at 93.472 196.088 0)
+      (effects (font (size 1.27 1.27)) hide)
+    )
+    (property "Datasheet" "" (id 3) (at 93.472 196.088 0)
+      (effects (font (size 1.27 1.27)) hide)
+    )
+    (pin "1")
   )
   (symbol (lib_id "Connector:USB_C_Plug_USB2.0") (at 148.082 45.212 0) (unit 1)
@@
     (pin "S1")
   )
-  (symbol (lib_id "Switch:SW_SPST") (at 138.176 94.742 0) (unit 1)
-    (in_bom yes) (on_board yes) (fields_autoplaced)
-    (property "Reference" "SW1" (id 0) (at 138.176 89.3912 0))
-    (property "Value" "SW_SPST" (id 1) (at 138.176 91.9281 0))
-    (property "Footprint" "" (id 2) (at 138.176 94.742 0)
-      (effects (font (size 1.27 1.27)) hide)
-    )
-    (property "Datasheet" "~" (id 3) (at 138.176 94.742 0)
+  (symbol (lib_id "Device:R") (at 93.472 192.278 180) (unit 1)
+    (in_bom yes) (on_board yes) (fields_autoplaced)
+    (property "Reference" "R18" (id 0) (at 95.25 191.4433 0)
+      (effects (font (size 1.27 1.27)) (justify right))
+    )
+    (property "Value" "0" (id 1) (at 95.25 193.9802 0)
+      (effects (font (size 1.27 1.27)) (justify right))
+    )
+    (property "Footprint" "Resistor_SMD:R_0402_1005Metric" (id 2) (at 95.25 192.278 90)
+      (effects (font (size 1.27 1.27)) hide)
+    )
+    (property "Datasheet" "~" (id 3) (at 93.472 192.278 0)
       (effects (font (size 1.27 1.27)) hide)
     )
@@
     (pin "1")
   )
+  (symbol (lib_id "New_Library:EG1206A") (at 153.162 109.22 0) (unit 1)
+    (in_bom yes) (on_board yes)
+    (property "Reference" "SW1" (id 0) (at 148.082 104.394 0))
+    (property "Value" "EG1206A" (id 1) (at 159.258 104.14 0))
+    (property "Footprint" "Library:EG1206A_EWI" (id 2) (at 153.162 101.6 0)
+      (effects (font (size 1.27 1.27)) hide)
+    )
+    (property "Datasheet" "" (id 3) (at 153.162 101.6 0)
+      (effects (font (size 1.27 1.27)) hide)
+    )
+    (pin "1")
+    (pin "2")
+    (pin "3")
+    (pin "4")
+    (pin "5")
+  )
+  (symbol (lib_id "power:GND") (at 93.472 178.308 90) (unit 1)
+    (in_bom yes) (on_board yes) (fields_autoplaced)
+    (property "Reference" "#PWR0149" (id 0) (at 99.822 178.308 0)
+      (effects (font (size 1.27 1.27)) hide)
+    )
+    (property "Value" "GND" (id 1) (at 96.647 178.7418 90)
+      (effects (font (size 1.27 1.27)) (justify right))
+    )
+    (property "Footprint" "" (id 2) (at 93.472 178.308 0)
+      (effects (font (size 1.27 1.27)) hide)
+    )
+    (property "Datasheet" "" (id 3) (at 93.472 178.308 0)
+      (effects (font (size 1.27 1.27)) hide)
+    )
+    (pin "1")
+  )
   (symbol (lib_id "Device:C") (at 265.938 113.03 0) (unit 1)
     (in_bom yes) (on_board yes) (fields_autoplaced)
@@
     (pin "1")
   )
-  (symbol (lib_id "power:GND") (at 84.836 113.284 0) (unit 1)
-    (in_bom yes) (on_board yes) (fields_autoplaced)
-    (property "Reference" "#PWR0137" (id 0) (at 84.836 119.634 0)
-      (effects (font (size 1.27 1.27)) hide)
-    )
-    (property "Value" "GND" (id 1) (at 84.836 117.7274 0))
-    (property "Footprint" "" (id 2) (at 84.836 113.284 0)
-      (effects (font (size 1.27 1.27)) hide)
-    )
-    (property "Datasheet" "" (id 3) (at 84.836 113.284 0)
-      (effects (font (size 1.27 1.27)) hide)
-    )
-    (pin "1")
+  (symbol (lib_id "Device:R") (at 93.472 182.118 0) (unit 1)
+    (in_bom yes) (on_board yes) (fields_autoplaced)
+    (property "Reference" "R17" (id 0) (at 95.25 181.2833 0)
+      (effects (font (size 1.27 1.27)) (justify left))
+    )
+    (property "Value" "0" (id 1) (at 95.25 183.8202 0)
+      (effects (font (size 1.27 1.27)) (justify left))
+    )
+    (property "Footprint" "Resistor_SMD:R_0402_1005Metric" (id 2) (at 91.694 182.118 90)
+      (effects (font (size 1.27 1.27)) hide)
+    )
+    (property "Datasheet" "~" (id 3) (at 93.472 182.118 0)
+      (effects (font (size 1.27 1.27)) hide)
+    )
+    (pin "1")
+    (pin "2")
   )
   (symbol (lib_id "Device:R") (at 224.79 102.108 90) (unit 1)
@@
     (pin "2")
   )
+  (symbol (lib_id "Device:R") (at 97.282 188.468 90) (unit 1)
+    (in_bom yes) (on_board yes) (fields_autoplaced)
+    (property "Reference" "R20" (id 0) (at 97.282 183.7522 90))
+    (property "Value" "0" (id 1) (at 97.282 186.2891 90))
+    (property "Footprint" "Resistor_SMD:R_0402_1005Metric" (id 2) (at 97.282 190.246 90)
+      (effects (font (size 1.27 1.27)) hide)
+    )
+    (property "Datasheet" "~" (id 3) (at 97.282 188.468 0)
+      (effects (font (size 1.27 1.27)) hide)
+    )
+    (pin "1")
+    (pin "2")
+  )
   (symbol (lib_id "Device:LED") (at 77.47 89.662 0) (unit 1)
     (in_bom yes) (on_board yes) (fields_autoplaced)
     (property "Reference" "D1" (id 0) (at 75.8825 84.6922 0))
     (property "Value" "LED" (id 1) (at 75.8825 87.2291 0))
-    (property "Footprint" "" (id 2) (at 77.47 89.662 0)
+    (property "Footprint" "LED_SMD:LED_0603_1608Metric" (id 2) (at 77.47 89.662 0)
       (effects (font (size 1.27 1.27)) hide)
     )
@@
     (property "Reference" "L1" (id 0) (at 252.73 87.7402 90))
     (property "Value" "2.2u" (id 1) (at 252.73 90.2771 90))
-    (property "Footprint" "" (id 2) (at 252.73 91.948 0)
+    (property "Footprint" "Inductor_SMD:L_0805_2012Metric" (id 2) (at 252.73 91.948 0)
       (effects (font (size 1.27 1.27)) hide)
     )
     (property "Datasheet" "~" (id 3) (at 252.73 91.948 0)
+      (effects (font (size 1.27 1.27)) hide)
+    )
+    (property "P/N" "74479775222A" (id 4) (at 252.73 91.948 90)
+      (effects (font (size 1.27 1.27)) hide)
+    )
+    (pin "1")
+    (pin "2")
+  )
+  (symbol (lib_id "Device:R") (at 97.282 185.928 90) (unit 1)
+    (in_bom yes) (on_board yes) (fields_autoplaced)
+    (property "Reference" "R19" (id 0) (at 97.282 181.2122 90))
+    (property "Value" "0" (id 1) (at 97.282 183.7491 90))
+    (property "Footprint" "Resistor_SMD:R_0402_1005Metric" (id 2) (at 97.282 187.706 90)
+      (effects (font (size 1.27 1.27)) hide)
+    )
+    (property "Datasheet" "~" (id 3) (at 97.282 185.928 0)
       (effects (font (size 1.27 1.27)) hide)
     )
@@
     (pin "2")
   )
-  (symbol (lib_id "Connector:Conn_01x02_Male") (at 79.756 110.744 0) (unit 1)
+  (symbol (lib_id "Connector:Conn_01x02_Male") (at 88.392 185.928 0) (unit 1)
     (in_bom yes) (on_board yes)
-    (property "Reference" "J8" (id 0) (at 80.391 106.968 0))
-    (property "Value" "Conn_01x02_Male" (id 1) (at 78.486 111.506 90))
-    (property "Footprint" "" (id 2) (at 79.756 110.744 0)
-      (effects (font (size 1.27 1.27)) hide)
-    )
-    (property "Datasheet" "~" (id 3) (at 79.756 110.744 0)
-      (effects (font (size 1.27 1.27)) hide)
-    )
+    (property "Reference" "J8" (id 0) (at 89.027 182.152 0))
+    (property "Value" "Conn_01x02_Male" (id 1) (at 87.122 186.69 90))
+    (property "Footprint" "Connector_JST:JST_PH_B2B-PH-K_1x02_P2.00mm_Vertical" (id 2) (at 88.392 185.928 0)
+      (effects (font (size 1.27 1.27)) hide)
+    )
+    (property "Datasheet" "~" (id 3) (at 88.392 185.928 0)
+      (effects (font (size 1.27 1.27)) hide)
+    )
