File: EE/Main/MainBoard/Power.kicad_sch (KiCad schematic)
At the start: 19 parts, among them J8 Conn_01x02_Male, P1 USB_C_Plug_USB2.0, SW1 EG1206A, U4 MCP73832-2-OT, U5 TPS62172DSG

Commit message: Routine Update
Parts:
- R14: value 20k -> 10k
Other:
- note added: "1000V/10,000 = 100mA"
- note removed: "1000V/20,000 = 50mA"
Changed lines of the file:
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@@
     (stroke (width 0) (type default) (color 0 0 0 0))
   )
-  (text "1000V/20,000 = 50mA" (at 25.908 106.68 0)
+  (text "1000V/10,000 = 100mA" (at 25.908 106.68 0)
     (effects (font (size 1.27 1.27)) (justify left bottom))
   )
@@
       (effects (font (size 1.27 1.27)) (justify left))
     )
-    (property "Value" "20k" (id 1) (at 40.386 96.774 90)
-      (effects (font (size 1.27 1.27)) (justify left))
-    )
+    (property "Value" "10k" (id 1) (at 40.386 96.774 90)
+      (effects (font (size 1.27 1.27)) (justify left))
+    )

Commit message: Random Check in
Parts:
- removed R16: 100k, Resistor_SMD:R_0402_1005Metric, symbol Device:R
- removed R17, R20: 0, Resistor_SMD:R_0402_1005Metric, symbol Device:R
- removed U5: TPS62172DSG, Package_SON:WSON-8-1EP_2x2mm_P0.5mm_EP0.9x1.6mm_ThermalVias, symbol Regulator_Switching:TPS62172DSG
- added C11, C12, C8: 4.7u, Capacitor_SMD:C_0603_1608Metric, symbol Device:C
- added L2: u, Inductor_SMD:L_0805_2012Metric, symbol Device:L
- added R4: 250m, Resistor_SMD:R_0805_2012Metric, symbol Device:R
- added R5: 0, Resistor_SMD:R_0402_1005Metric_Pad0.72x0.64mm_HandSolder, symbol Device:R
- added R6, R7: R, symbol Device:R
- added TP+, TP-, TPVBAT, TPVBUS, TPVCC, TPVd: TestPoint, TestPoint:TestPoint_Pad_1.5x1.5mm, symbol Connector:TestPoint
- added U2: LM3670MF-3.3, Package_TO_SOT_SMD:TSOT-23-5, symbol Regulator_Switching:LM3670MF
- added U5: MCP1640Cx-xCHY, Package_TO_SOT_SMD:SOT-23-6, symbol Regulator_Switching:MCP1640Cx-xCHY
- L1: value 2.2u -> 10u
Connections:
- net GND: now also C11.2, C12.2, C8.2, R6.2, U2.2 (GND), U5.2 (GND)
- net VBAT: now also R4.2, TP+.1, TPVBAT.1
- net VBUS: now also TPVBUS.1
- net VCC: now also C8.1, TPVCC.1, U2.4 (FB), U5.3 (EN), U5.6 (V_{IN})
- net V_PRE_REG: now also R5.1, U2.1 (Vin), U2.3 (EN); no longer SW1.2 (COM)
- net at SW1.3: now also R4.1, TP-.1
- net at L1.1: now also U2.5 (SW)
- new net: R5.2, SW1.2 (COM)
- new net: R6.1, R7.2, U5.4 (V_{FB})
- new net Vdrive: C11.1, C12.1, L2.2, TPVd.1
- no-connect marks 8 -> 7
Other:
- note added: "Regulators"
- note added: "TODO Need to boost back up to 3.9V"
- note added: "TODO double check schematic"
- note added: "TODO math for resistors"
- note removed: "GND because fixed output @ 3.3V"
- note removed: "Regulator"
- moved on the sheet: C4, C5, C6, J8, L1, R18, R19, SW1
