File: EE/Main/MainBoard/Power.kicad_sch (KiCad schematic)
At the start: 39 parts, among them J8 Conn_01x02_Male, P1 USB_C_Plug_USB2.0, Q1 Q_PMOS_GSD, Q2 Q_NMOS_GSD, SW1 SW_DPST, U2 MCP73832-2-OT, U5 LM3670MF-3.3

Commit message: Potential Revision
Potentially fabb-able rev.
Parts:
- removed C11, C5: 4.7u, Capacitor_SMD:C_0603_1608Metric, symbol Device:C
- removed L1: 0.47u, Inductor_SMD:L_0805_2012Metric, symbol Device:L
- removed R18: 10K, Resistor_SMD:R_0402_1005Metric, symbol Device:R
- removed R21, R22: 10k, Resistor_SMD:R_0402_1005Metric, symbol Device:R
- removed R23: 550k, Resistor_SMD:R_0402_1005Metric, symbol Device:R
- removed R24: 100k, Resistor_SMD:R_0402_1005Metric, symbol Device:R
- removed R26: 1M, Resistor_SMD:R_0402_1005Metric, symbol Device:R
- removed TP3v1: TestPoint, TestPoint:TestPoint_Pad_1.5x1.5mm, symbol Connector:TestPoint
- removed U4: ~, Package_TO_SOT_SMD:SOT-583-8, symbol library:TPS61033
Connections:
- net GND: now also P1.S1 (SHIELD)
- no-connect marks 5 -> 4
Other:
- note added: "Thought process: VBAT has only R6 as a drain source. Once the button is pressed, the Fet turns on enabling power to go through VBAT_OUT goes to power the 3v3 buck rail. Once 3v3 is enabled, the pull up will maintain through R15, and the MCU can turn itself off by pulling the gate low"
- note removed: "Momentary button MCU will hold on Remove parallel resistor to switch on release."
- note removed: "R20= (Vout/vref-1)*R19 R20= (3.9/0.6-1)*100k R20 = 550k"
- note removed: "Thought process: VBAT has only R6 as a drain source. Once the button is pressed, the Fet turns on enabling power to go through VBAT_OUT goes to power the 3v3 buck rail. Once 3v3 is eenabled, the pull up will maintain through R15, and the MCU can turn itself off by pulling the gate low"
- moved on the sheet: Q2, R12, R13, R14, R15, R6, TP+1, TP-1, TPPGate1

Commit message: Updated EE
Parts:
- R13: value 10k_NP -> 100k
Other:
- note added: "TODO does R15 need to migrate to 1M?"
- note added: "TODO is R13 Necessary to stay off?"
- note added: "TODO this appears broken"
Changed lines of the file:
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@@
+		)
+	)
+	(text "TODO this appears broken"
+		(exclude_from_sim no)
+		(at 170.434 61.468 90)
+		(effects
+			(font
+				(size 1.27 1.27)
+			)
+		)
+	)
+	(text "TODO does R15 need to migrate to 1M?"
+		(exclude_from_sim no)
+		(at 86.106 71.882 0)
+		(effects
+			(font
+				(size 1.27 1.27)
+			)
+		)
+	)
+	(text "TODO is R13 Necessary to stay off?"
+		(exclude_from_sim no)
+		(at 86.106 74.676 0)
+		(effects
+			(font
+				(size 1.27 1.27)
+			)
 		)
 	)
@@
 		)
 	)
-	(label "N_GATE"
-		(at 266.7 19.05 180)
-		(fields_autoplaced yes)
+	(text "TODO this appears broken"
+		(exclude_from_sim no)
+		(at 247.65 119.38 0)
 		(effects
 			(font
 				(size 1.27 1.27)
 			)
-			(justify right bottom)
-		)
-	)
-	(label "VBAT_OUT"
-		(at 233.68 127 180)
+		)
+	)
+	(label "N_GATE"
+		(at 266.7 19.05 180)
 		(fields_autoplaced yes)
 		(effects
@@
 		)
 	)
-	(label "BTN_SNS"
-		(at 152.4 81.28 270)
+	(label "VBAT_OUT"
+		(at 233.68 127 180)
 		(fields_autoplaced yes)
 		(effects
@@
 		)
 	)
-	(label "N_GATE"
-		(at 114.3 83.82 180)
+	(label "BTN_SNS"
+		(at 152.4 81.28 270)
 		(fields_autoplaced yes)
 		(effects
@@
 		)
 	)
-	(label "VBAT"
-		(at 138.43 55.88 180)
+	(label "N_GATE"
+		(at 114.3 83.82 180)
 		(fields_autoplaced yes)
 		(effects
@@
 		)
 	)
-	(label "P_DRAIN"
-		(at 138.43 39.37 180)
+	(label "VBAT"
+		(at 138.43 55.88 180)
 		(fields_autoplaced yes)
 		(effects
@@
 		)
 	)
-	(label "VBAT_OUT"
-		(at 161.29 39.37 0)
+	(label "P_DRAIN"
+		(at 138.43 39.37 180)
 		(fields_autoplaced yes)
 		(effects
@@
 				(size 1.27 1.27)
 			)
-			(justify left bottom)
+			(justify right bottom)
 		)
 	)
 	(label "VBAT_OUT"
-		(at 266.7 15.24 180)
+		(at 161.29 39.37 0)
 		(fields_autoplaced yes)
 		(effects
@@
 				(size 1.27 1.27)
 			)
-			(justify right bottom)
-		)
-	)
-	(label "VBAT"
-		(at 109.22 177.8 270)
+			(justify left bottom)
+		)
+	)
+	(label "VBAT_OUT"
+		(at 266.7 15.24 180)
 		(fields_autoplaced yes)
 		(effects
@@
 	)
 	(label "VBAT"
-		(at 140.97 63.5 180)
+		(at 109.22 177.8 270)
 		(fields_autoplaced yes)
 		(effects
@@
 		)
 	)
-	(label "N_SOURCE"
-		(at 125.73 95.25 180)
+	(label "VBAT"
+		(at 140.97 63.5 180)
 		(fields_autoplaced yes)
 		(effects
@@
 		)
 	)
-	(label "VBAT"
-		(at 73.152 170.688 0)
+	(label "N_SOURCE"
+		(at 125.73 95.25 180)
 		(fields_autoplaced yes)
 		(effects
@@
 				(size 1.27 1.27)
 			)
-			(justify left bottom)
-		)
-	)
-	(label "BTN_SNS"
-		(at 266.7 22.86 180)
+			(justify right bottom)
+		)
+	)
+	(label "VBAT"
+		(at 73.152 170.688 0)
 		(fields_autoplaced yes)
 		(effects
@@
 				(size 1.27 1.27)
 			)
+			(justify left bottom)
+		)
+	)
+	(label "BTN_SNS"
+		(at 266.7 22.86 180)
+		(fields_autoplaced yes)
+		(effects
+			(font
+				(size 1.27 1.27)
+			)
 			(justify right bottom)
 		)
@@
 			)
 		)
-		(property "Value" "10k_NP"
+		(property "Value" "100k"
 			(at 110.998 92.6521 0)
 			(effects
