File: EE/Main/MainBoard/mcu.kicad_sch (KiCad schematic)
At the start: 0 parts

Commit message: Updated layout, and placement for main board
Parts:
- added C1: 0.1u, Capacitor_SMD:C_0402_1005Metric, symbol Device:C
- added J7: TAG_CONNECT, Connector:Tag-Connect_TC2030-IDC-FP_2x03_P1.27mm_Vertical, symbol ACTempDisconnect:TAG_CONNECT
- added R1, R2: 4.7k, Resistor_SMD:R_0402_1005Metric, symbol Device:R
- added U1: STM32C011F4U6TR, Package_DFN_QFN:UQFN-20_3x3mm_P0.4mm, symbol New_Library:STM32C011F4U6TR
Connections:
- new net A_EN: U1.5 (PA0)
- new net B_EN: U1.6 (PA1)
- new net C_EN: U1.7 (PA2)
- new net D1_G_EN: U1.14 (PA11_9)
- new net D1_R_EN: U1.12 (PA7)
- new net D2_G_EN: U1.15 (PA12_10)
- new net D2_R_EN: U1.13 (PA8)
- new net D_EN: U1.8 (PA3)
- new net E_EN: U1.9 (PA4)
- new net F_EN: U1.10 (PA5)
- new net GND: C1.2, J7.3 (GND), U1.3 (VSS_A)
- new net G_EN: U1.11 (PA6)
- new net SCL: R2.2, U1.18 (PB6)
- new net SDA: R1.2, U1.19 (PB7)
- new net SWDCLK: J7.5 (SWCLK), U1.17 (PA14_B0)
- new net SWDIO: J7.6 (SWDIO), U1.16 (PA13)
- new net VCC: C1.1, J7.1 (POWER_3V3), R1.1, R2.1, U1.2 (VDD_A)
- no-connect marks 0 -> 5

Commit message: Routed PCB, Need SCL/SDA still
Connections:
- net A_EN: now also U1.11 (PA6); no longer U1.5 (PA0)
- net B_EN: now also U1.13 (PA8); no longer U1.6 (PA1)
- net C_EN: now also U1.9 (PA4); no longer U1.7 (PA2)
- net D1_G_EN: now also U1.6 (PA1); no longer U1.14 (PA11_9)
- net D1_R_EN: now also U1.15 (PA12_10); no longer U1.12 (PA7)
- net D2_G_EN: now also U1.5 (PA0); no longer U1.15 (PA12_10)
- net D2_R_EN: now also U1.14 (PA11_9); no longer U1.13 (PA8)
- net D_EN: now also U1.7 (PA2); no longer U1.8 (PA3)
- net E_EN: now also U1.8 (PA3); no longer U1.9 (PA4)
- net F_EN: now also U1.12 (PA7); no longer U1.10 (PA5)
- net G_EN: now also U1.10 (PA5); no longer U1.11 (PA6)
Changed lines of the file:
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@@
   (no_connect (at 52.07 143.256))
   (no_connect (at 52.07 148.336))
-  (no_connect (at 157.734 75.946))
   (no_connect (at 157.734 78.486))
   (no_connect (at 157.734 81.026))
+  (no_connect (at 157.734 75.946))
   (wire (pts (xy 63.246 145.796) (xy 63.246 146.558))
     (stroke (width 0) (type default) (color 0 0 0 0))
@@
     (effects (font (size 1.27 1.27)) (justify right bottom))
   )
-  (label "D1_G_EN" (at 129.794 79.756 180)
-    (effects (font (size 1.27 1.27)) (justify right bottom))
-  )
   (label "SCL" (at 189.23 58.928 270)
     (effects (font (size 1.27 1.27)) (justify right bottom))
@@
     (effects (font (size 1.27 1.27)) (justify left bottom))
   )
+  (label "D1_G_EN" (at 129.794 59.436 180)
+    (effects (font (size 1.27 1.27)) (justify right bottom))
+  )
   (label "G_EN" (at 274.32 29.464 180)
     (effects (font (size 1.27 1.27)) (justify right bottom))
@@
     (effects (font (size 1.27 1.27)) (justify right bottom))
   )
-  (label "D2_G_EN" (at 129.794 82.296 180)
+  (label "SDA" (at 183.642 58.928 270)
     (effects (font (size 1.27 1.27)) (justify right bottom))
   )
-  (label "SDA" (at 183.642 58.928 270)
+  (label "B_EN" (at 129.794 77.216 180)
     (effects (font (size 1.27 1.27)) (justify right bottom))
   )
@@
     (effects (font (size 1.27 1.27)) (justify right bottom))
   )
+  (label "D1_R_EN" (at 129.794 82.296 180)
+    (effects (font (size 1.27 1.27)) (justify right bottom))
+  )
   (label "SCL" (at 17.526 18.034 0)
     (effects (font (size 1.27 1.27)) (justify left bottom))
   )
-  (label "A_EN" (at 129.794 56.896 180)
+  (label "D2_R_EN" (at 129.794 79.756 180)
+    (effects (font (size 1.27 1.27)) (justify right bottom))
+  )
+  (label "A_EN" (at 129.794 72.136 180)
+    (effects (font (size 1.27 1.27)) (justify right bottom))
+  )
+  (label "G_EN" (at 129.794 69.596 180)
     (effects (font (size 1.27 1.27)) (justify right bottom))
   )
@@
     (effects (font (size 1.27 1.27)) (justify left bottom))
   )
-  (label "F_EN" (at 129.794 69.596 180)
+  (label "D2_G_EN" (at 129.794 56.896 180)
     (effects (font (size 1.27 1.27)) (justify right bottom))
   )
@@
     (effects (font (size 1.27 1.27)) (justify right bottom))
   )
-  (label "D2_R_EN" (at 129.794 77.216 180)
-    (effects (font (size 1.27 1.27)) (justify right bottom))
-  )
   (label "E_EN" (at 274.32 24.384 180)
     (effects (font (size 1.27 1.27)) (justify right bottom))
   )
-  (label "D1_R_EN" (at 129.794 74.676 180)
+  (label "D2_G_EN" (at 274.32 39.37 180)
     (effects (font (size 1.27 1.27)) (justify right bottom))
   )
-  (label "E_EN" (at 129.794 67.056 180)
-    (effects (font (size 1.27 1.27)) (justify right bottom))
-  )
-  (label "C_EN" (at 129.794 61.976 180)
-    (effects (font (size 1.27 1.27)) (justify right bottom))
-  )
-  (label "D2_G_EN" (at 274.32 39.37 180)
+  (label "F_EN" (at 129.794 74.676 180)
     (effects (font (size 1.27 1.27)) (justify right bottom))
   )
@@
     (effects (font (size 1.27 1.27)) (justify right bottom))
   )
-  (label "D_EN" (at 129.794 64.516 180)
+  (label "E_EN" (at 129.794 64.516 180)
+    (effects (font (size 1.27 1.27)) (justify right bottom))
+  )
+  (label "C_EN" (at 129.794 67.056 180)
     (effects (font (size 1.27 1.27)) (justify right bottom))
   )
@@
     (effects (font (size 1.27 1.27)) (justify right bottom))
   )
-  (label "G_EN" (at 129.794 72.136 180)
+  (label "D_EN" (at 129.794 61.976 180)
     (effects (font (size 1.27 1.27)) (justify right bottom))
   )
@@
     (effects (font (size 1.27 1.27)) (justify left bottom))
   )
-  (label "B_EN" (at 129.794 59.436 180)
-    (effects (font (size 1.27 1.27)) (justify right bottom))
-  )
   (hierarchical_label "SDA" (shape input) (at 17.526 15.494 180)
