File: EE/Main/MainBoard/MainBoard.kicad_pcb (KiCad board)
At the start: 2 copper layers, 140.8 x 87.5 mm, 107 parts, among them J1 Conn_01x04_Male, J2 Conn_01x04_Male, J3 Conn_01x04_Male, J4 Conn_01x04_Male, J5 Conn_01x04_Male, J6 Conn_01x04_Male, J7 TAG_CONNECT, J8 Conn_01x02_Male, J9 Conn_01x04_Male, P1 USB_C_Plug_USB2.0, Q1 Q_PMOS_GSD, Q2 Q_NMOS_GSD, SW1 SW_DPST, U1 STM32G431K6Tx, U10 DRV5032AJDBZR, U2 MCP73832-2-OT, U3 SN74LVC1T45DBV, U5 LM3670MF-3.3, U6 DRV5032AJDBZR, U7 DRV5032AJDBZR, U8 DRV5032AJDBZR, U9 DRV5032AJDBZR, Y1 Crystal

Commit message: Potential Revision
Potentially fabb-able rev.
Parts:
- removed the C5 at (143.7, 105.4)
- removed the C5 at (152.6, 122.5)
- removed the C6 at (152.6, 123.9)
- removed L1: 0.47u, Inductor_SMD:L_0805_2012Metric
- removed R17, R19, R24: 100k, Resistor_SMD:R_0402_1005Metric
- removed R18: 10K, Resistor_SMD:R_0402_1005Metric
- removed R21, R22: 10k, Resistor_SMD:R_0402_1005Metric
- removed R23: 550k, Resistor_SMD:R_0402_1005Metric
- removed R26: 1M, Resistor_SMD:R_0402_1005Metric
- removed TP3v1, TPDIN1, TP_DIN_UP1: TestPoint, TestPoint:TestPoint_Pad_1.5x1.5mm
- removed the TPVCC1 at (153.8, 126.3)
- removed U3: SN74LVC1T45DBV, Package_TO_SOT_SMD:SOT-23-6
- removed U4: ~, Package_TO_SOT_SMD:SOT-583-8
- added C5: C_NP, Capacitor_SMD:C_0402_1005Metric_Pad0.74x0.62mm_HandSolder, F.Cu at (199.5, 73.3)
- added D2: LED, LED_SMD:LED_0603_1608Metric, F.Cu at (121.4, 65.1)
- added H13: MountingHole, MountingHole:MountingHole_2.7mm, F.Cu at (110.2, 112.0)
- added H14: MountingHole, MountingHole:MountingHole_2.7mm, F.Cu at (164.8, 71.3)
- added H15: MountingHole, MountingHole:MountingHole_2.7mm, F.Cu at (185.2, 98.0)
- added R20: 4.7k, Resistor_SMD:R_0402_1005Metric, F.Cu at (119.3, 63.0)
- C10, C9: value 0.1u -> C_NP; footprint Capacitor_SMD:C_0402_1005Metric -> Capacitor_SMD:C_0402_1005Metric_Pad0.74x0.62mm_HandSolder
- C11: value 4.7u -> C_NP; footprint Capacitor_SMD:C_0603_1608Metric -> Capacitor_SMD:C_0402_1005Metric_Pad0.74x0.62mm_HandSolder
- J9: value Conn_01x04_Male -> Conn_01x06
- P1: moved to B.Cu
- moved TPVCC1 69.3 mm to (185.8, 113.8), turned to 0 degrees
- moved P1 69.0 mm to (178.4, 132.7), turned to 180 degrees
- moved R25 67.0 mm to (185.3, 116.4), turned to -90 degrees
- moved L2 66.6 mm to (183.3, 113.1), turned to -90 degrees
- moved C9 66.2 mm to (193.6, 108.7), turned to 45 degrees
- moved TPVBUS1 65.1 mm to (177.5, 126.7), turned to 90 degrees
- moved C8 65.1 mm to (183.8, 116.4), turned to -90 degrees
- moved U5 62.9 mm to (180.2, 113.1), turned to 0 degrees
- moved C6 62.5 mm to (181.8, 116.4), turned to -90 degrees
- moved C2 60.4 mm to (174.8, 123.8), turned to 90 degrees
- moved C4 59.0 mm to (177.4, 113.8), turned to 90 degrees
- moved C10 53.9 mm to (171.0, 60.8), turned to -90 degrees
- moved R14 50.2 mm to (157.6, 116.3)
- moved R6 50.2 mm to (161.3, 114.1)
- moved TP-1 50.2 mm to (169.9, 111.8)
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Connections:
- C10 pad 1: Vdrive -> /SCL
- C11 pad 1: Vdrive -> /SDA
- C9 pad 2: GND -> /SDA
- J9 pad 2: Vdrive -> +3V3
- J9 pad 3: /Display/DISPLAY_DIN -> unconnected-(J9-Pin_3-Pad3)
- P1 pad S1: unconnected-(P1-SHIELD-PadS1)_3 -> GND
- U1 pad 10: unconnected-(U1-PA5-Pad10) -> /Display/DISPLAY_CIN
- U1 pad 11: unconnected-(U1-PA6-Pad11) -> /MCU/End
- U1 pad 12: /MCU/N_GATE -> /Display/DISPLAY_DIN
- U1 pad 13: /MCU/BTN_SNS -> /MCU/ADC
- U1 pad 18: /SDA -> /MCU/N_GATE
- U1 pad 19: /SCL -> unconnected-(U1-PA9-Pad19)
- U1 pad 25: /MCU/End -> /SCL
- U1 pad 26: /MCU/Start_00 -> /MCU/HB
- U1 pad 27: /MCU/Start_01 -> unconnected-(U1-PB4-Pad27)
- U1 pad 28: /MCU/Start_11 -> unconnected-(U1-PB5-Pad28)
- U1 pad 29: /MCU/Start_10 -> unconnected-(U1-PB6-Pad29)
- U1 pad 30: /MCU/DISPLAY_DIN -> /SDA
- U1 pad 5: /MCU/ADC -> /MCU/Start_00
- U1 pad 6: unconnected-(U1-PA1-Pad6) -> /MCU/Start_01
- U1 pad 7: unconnected-(U1-PA2-Pad7) -> /MCU/Start_10
- U1 pad 8: /MCU/DISP_EN -> /MCU/Start_11
- U1 pad 9: unconnected-(U1-PA4-Pad9) -> /MCU/BTN_SNS
Routing:
- net Vdrive: track 61.2 -> 0.00 mm, vias 3 -> 0
- net /MCU/DISP_EN: track 57.9 -> 0.00 mm
- net VBUS: track 81.1 -> 30.6 mm, vias 4 -> 0
- net Net-(Q1-G): track 70.3 -> 26.6 mm
- net +3V3: track 748.1 -> 711.8 mm, vias 14 -> 7
- net /Power/VBAT: track 78.0 -> 44.4 mm, vias 2 -> 0
- net /MCU/End: track 38.9 -> 65.8 mm
- net /MCU/BTN_SNS: track 71.2 -> 46.3 mm
- net /MCU/N_GATE: track 77.8 -> 59.4 mm
- net /MCU/DISPLAY_DIN: track 17.9 -> 0.00 mm
- net /Display/DISPLAY_CIN: track 0.00 -> 14.2 mm
- net /MCU/DIR: track 12.2 -> 0.00 mm
- net /SCL: track 289.9 -> 296.6 mm, vias 2 -> 4
- net /MCU/ADC_: track 85.4 -> 79.1 mm, vias 4 -> 2
- net /MCU/HB: track 0.00 -> 5.50 mm
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- added copper zone on F.Cu, net +3V3
Other:
- board text added: "Direction"
- board text added: "Start"

Commit message: Checkin of Fabbed Board
Routing:
- net GND: track 65.7 -> 68.2 mm, vias 350 -> 349
Changed lines of the file:
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@@
 		(tags "resistor")
 		(property "Reference" "R10"
-			(at 0 -1.17 0)
+			(at 0.375 -1.45 0)
 			(layer "F.SilkS")
 			(effects
@@
 		(tags "TSOT TO_SOT_SMD")
 		(property "Reference" "U5"
-			(at 0 -2.4 360)
+			(at 0 -2.4 0)
 			(layer "F.SilkS")
 			(effects
@@
 		)
 		(property "Value" "LM3670MF-3.3"
-			(at 0 2.4 360)
+			(at 0 2.4 0)
 			(layer "F.Fab")
 			(effects
@@
 		)
 		(fp_text user "${REFERENCE}"
-			(at 0 0 360)
+			(at 0 0 0)
 			(layer "F.Fab")
 			(effects
@@
 		(tags "capacitor")
 		(property "Reference" "C8"
-			(at 1.953 -1.5285 360)
+			(at 1.953 -1.5285 0)
 			(layer "F.SilkS")
 			(effects
@@
 		)
 		(property "Value" "TestPoint"
-			(at 0 1.75 360)
+			(at 0 1.75 0)
 			(layer "F.Fab")
 			(effects
@@
 		)
 		(fp_text user "${REFERENCE}"
-			(at 0 -1.65 360)
+			(at 0 -1.65 0)
 			(layer "F.Fab")
 			(effects
@@
 		(tags "capacitor")
 		(property "Reference" "C6"
-			(at 2.032 0 360)
+			(at 2.032 0 0)
 			(layer "F.SilkS")
 			(effects
@@
 		(tags "LED")
 		(property "Reference" "D1"
-			(at 0 -1.43 360)
+			(at 0 -1.43 0)
 			(layer "F.SilkS")
 			(effects
@@
 		)
 		(property "Value" "LED"
-			(at 0 1.43 360)
+			(at 0 1.43 0)
 			(layer "F.Fab")
 			(effects
@@
 		)
 		(fp_text user "${REFERENCE}"
-			(at 0 0 360)
+			(at 0 0 0)
 			(layer "F.Fab")
 			(effects
@@
 		(tags "resistor")
 		(property "Reference" "R5"
-			(at 0 -1.17 360)
+			(at 0 -1.17 0)
 			(layer "F.SilkS")
 			(effects
@@
 		)
 		(property "Value" "4.7k"
-			(at 0 1.17 360)
+			(at 0 1.17 0)
 			(layer "F.Fab")
 			(effects
@@
 		)
 		(fp_text user "${REFERENCE}"
-			(at 0 0 360)
+			(at 0 0 0)
 			(layer "F.Fab")
 			(effects
@@
 		(tags "SOT TO_SOT_SMD")
 		(property "Reference" "U8"
-			(at 0 -2.4 90)
+			(at 0.361 -2.657 90)
 			(layer "F.SilkS")
 			(effects
@@
 		(tags "resistor")
 		(property "Reference" "R25"
-			(at -0.066001 -1.0205 90)
+			(at -0.066001 -1.194 90)
 			(layer "F.SilkS")
 			(effects
@@
 		(tags "resistor")
 		(property "Reference" "R4"
-			(at 0 -1.17 360)
+			(at 0 -1.17 0)
 			(layer "F.SilkS")
 			(effects
@@
 		)
 		(property "Value" "10k"
-			(at 0 1.17 360)
+			(at 0 1.17 0)
 			(layer "F.Fab")
 			(effects
@@
 		)
 		(fp_text user "${REFERENCE}"
-			(at 0 0 360)
+			(at 0 0 0)
 			(layer "F.Fab")
 			(effects
@@
 		(tags "USB Type-C Receptacle Through-hole Right angle")
 		(property "Reference" "P1"
-			(at 2.975 1.8 360)
+			(at 2.975 1.8 0)
 			(layer "B.SilkS")
 			(effects
@@
 		)
 		(property "Value" "USB_C_Plug_USB2.0"
-			(at 2.975 -9.925 360)
+			(at 2.975 -9.925 0)
 			(layer "B.Fab")
 			(effects
@@
 		)
 		(fp_text user "PCB Edge"
-			(at 2.975 -6.1 360)
+			(at 2.975 -6.1 0)
 			(layer "Dwgs.User")
 			(effects
@@
 		)
 		(fp_text user "${REFERENCE}"
-			(at 2.975 -4.025 360)
+			(at 2.975 -4.025 0)
 			(layer "B.Fab")
 			(effects
@@
 		(effects
 			(font
-				(size 1 1)
-				(thickness 0.15)
+				(size 1.2 1.2)
+				(thickness 0.2)
+				(bold yes)
 			)
 			(justify left bottom)
@@
 	)
 	(gr_text "PRT-13851"
-		(at 144.525 87.529999 -90)
+		(at 143 80.78 0)
 		(layer "F.SilkS")
 		(effects
@@
 	)
 	(segment
-		(start 172.105 133.71)
-		(end 172.475 134.08)
-		(width 0.2)
-		(layer "F.Cu")
-		(net 1)
-	)
-	(segment
 		(start 108.325 101.855)
 		(end 108.325 100.895)
@@
 	)
 	(segment
-		(start 172.475 132.73)
-		(end 172.475 134.08)
-		(width 0.2)
-		(layer "F.Cu")
-		(net 1)
-	)
-	(segment
 		(start 160.585 88.365)
 		(end 160.5 88.28)
@@
 	)
 	(segment
-		(start 171.125 133.71)
-		(end 172.105 133.71)
-		(width 0.2)
-		(layer "F.Cu")
-		(net 1)
-	)
-	(segment
 		(start 185.306 116.885249)
 		(end 185.306 118.086)
@@
 	)
 	(via
-		(at 186.5 70.53)
-		(size 0.8)
-		(drill 0.4)
-		(layers "F.Cu" "B.Cu")
-		(net 1)
-	)
-	(via
 		(at 194 71.78)
 		(size 0.8)
@@
 	)
 	(segment
+		(start 171.495 134.08)
+		(end 171.125 133.71)
+		(width 0.2)
+		(layer "B.Cu")
+		(net 1)
+	)
+	(segment
+		(start 172.475 134.08)
+		(end 172.475 132.73)
+		(width 0.2)
+		(layer "B.Cu")
+		(net 1)
+	)
+	(segment
+		(start 172.475 134.08)
+		(end 172.475 135.505)
+		(width 0.2)
+		(layer "B.Cu")
+		(net 1)
+	)
+	(segment
+		(start 172.475 134.08)
+		(end 171.495 134.08)
+		(width 0.2)
+		(layer "B.Cu")
+		(net 1)
+	)
+	(segment
+		(start 178.425 134.08)
+		(end 178.425 135.205)
+		(width 0.2)
+		(layer "B.Cu")
+		(net 1)
+	)
+	(segment
 		(start 177.5125 126.705001)
 		(end 177.5125 131.707474)
@@
 	)
 	(segment
-		(start 128.146532 61.37545)
-		(end 127.376082 60.605)
-		(width 0.2)
-		(layer "F.Cu")
-		(net 30)
-	)
-	(segment
 		(start 208.2 78.68)
 		(end 206.2 76.88)
@@
 	)
 	(segment
+		(start 128.146532 63.062444)
+		(end 128 62.915912)
+		(width 0.2)
+		(layer "F.Cu")
+		(net 30)
+	)
+	(segment
 		(start 95.88941 95.823589)
 		(end 96.79941 96.733589)
@@
 	)
 	(segment
+		(start 128.341531 63.257445)
+		(end 128.146532 63.062444)
+		(width 0.2)
+		(layer "F.Cu")
+		(net 30)
+	)
+	(segment
 		(start 105.6 64.355)
 		(end 99.79 58.545)
@@
 	)
 	(segment
-		(start 101.95 90.58)
-		(end 101.88 90.58)
-		(width 0.2)
-		(layer "F.Cu")
-		(net 30)
-	)
-	(segment
 		(start 141 122.78)
 		(end 146.975 128.755)
@@
 	)
 	(segment
-		(start 128.146532 63.062444)
-		(end 128.146532 61.842465)
-		(width 0.2)
-		(layer "F.Cu")
-		(net 30)
-	)
-	(segment
 		(start 160.585 98.99)
 		(end 160.585 91.060001)
@@
 	)
 	(segment
+		(start 127.900541 61.129459)
+		(end 127.376082 60.605)
+		(width 0.2)
+		(layer "F.Cu")
+		(net 30)
+	)
+	(segment
 		(start 132.725 51.755)
 		(end 132.65 51.68)
@@
 	)
 	(segment
-		(start 128.341531 63.257445)
-		(end 128.146532 63.062444)
-		(width 0.2)
-		(layer "F.Cu")
-		(net 30)
-	)
-	(segment
 		(start 184.034 115.865251)
 		(end 183.782 115.61325)
@@
 	)
 	(segment
+		(start 128.341531 63.762445)
+		(end 128.341531 63.257445)
+		(width 0.2)
+		(layer "F.Cu")
+		(net 30)
+	)
+	(segment
 		(start 115.679248 61.266752)
 		(end 115.679248 65.584752)
@@
 	)
 	(segment
-		(start 128.146532 61.842465)
-		(end 128.146532 61.37545)
-		(width 0.2)
-		(layer "F.Cu")
-		(net 30)
-	)
-	(segment
 		(start 133.52 68.705)
 		(end 130.3475 71.8775)
@@
 	)
 	(segment
+		(start 128 61.228918)
+		(end 127.900541 61.129459)
+		(width 0.2)
+		(layer "F.Cu")
+		(net 30)
+	)
+	(segment
 		(start 73 83.08)
 		(end 73 106.68)
@@
 	)
 	(segment
+		(start 128 62.915912)
+		(end 128 61.228918)
+		(width 0.2)
+		(layer "F.Cu")
+		(net 30)
+	)
+	(segment
 		(start 185.306 115.86525)
 		(end 184.034 115.865251)
@@
 	)
 	(segment
-		(start 128.341531 63.762445)
-		(end 128.341531 63.257445)
-		(width 0.2)
-		(layer "F.Cu")
-		(net 30)
-	)
-	(segment
 		(start 183.537001 114.13575)
 		(end 183.8375 113.83525)
@@
 		(width 0.2)
 		(layer "F.Cu")
-		(net 30)
-	)
-	(segment
-		(start 128.146532 61.842465)
-		(end 128.146533 61.562445)
-		(width 0.2)
-		(layer "F.Cu")
