File: EE/Sensing/SensorBoard/SensorBoard.kicad_sch (KiCad schematic)
At the start: 23 parts, among them J1 Conn_01x04_Male, Q11 DMP31D1U-7, Q12 DMP31D1U-7, U1 TCR2EE27, U2 TCR2EE32, U3 TCA9555PWR

Commit message: Fixed Routing
Connections:
- net 2v7_EN: now also U3.10 (P06); no longer U3.4 (P00)
- net 3v2_EN: now also U3.19 (P16); no longer U3.5 (P01)
- net B00: now also U3.18 (P15); no longer U3.8 (P04)
- net B01: now also U3.17 (P14); no longer U3.9 (P05)
- net B02: now also U3.16 (P13); no longer U3.10 (P06)
- net B03: now also U3.15 (P12); no longer U3.11 (P07)
- net B04: now also U3.14 (P11); no longer U3.13 (P10)
- net B0_EN: now also U3.11 (P07); no longer U3.6 (P02)
- net B10: now also U3.13 (P10); no longer U3.14 (P11)
- net B11: now also U3.6 (P02); no longer U3.15 (P12)
- net B12: now also U3.7 (P03); no longer U3.16 (P13)
- net B13: now also U3.8 (P04); no longer U3.17 (P14)
- net B14: now also U3.9 (P05); no longer U3.18 (P15)
- net B1_EN: now also U3.20 (P17); no longer U3.7 (P03)
- net SCL: now also J1.2 (Pin_2); no longer J1.3 (Pin_3)
- net SDA: now also J1.3 (Pin_3); no longer J1.2 (Pin_2)
- net VCC: now also U3.24 (VCC)
Changed lines of the file:
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@@
     (effects (font (size 1.27 1.27)) (justify left bottom))
   )
-  (label "B12" (at 231.902 136.144 0)
-    (effects (font (size 1.27 1.27)) (justify left bottom))
-  )
-  (label "2v7_EN" (at 231.902 105.664 0)
+  (label "B10" (at 231.902 128.524 0)
     (effects (font (size 1.27 1.27)) (justify left bottom))
   )
@@
     (effects (font (size 1.27 1.27)) (justify right bottom))
   )
-  (label "B13" (at 231.902 138.684 0)
-    (effects (font (size 1.27 1.27)) (justify left bottom))
-  )
   (label "B02" (at 121.666 26.67 0)
+    (effects (font (size 1.27 1.27)) (justify left bottom))
+  )
+  (label "SDA" (at 257.81 33.274 0)
     (effects (font (size 1.27 1.27)) (justify left bottom))
   )
@@
     (effects (font (size 1.27 1.27)) (justify right bottom))
   )
-  (label "SCL" (at 257.81 33.274 0)
-    (effects (font (size 1.27 1.27)) (justify left bottom))
-  )
   (label "B11" (at 121.666 79.248 0)
-    (effects (font (size 1.27 1.27)) (justify left bottom))
-  )
-  (label "B00" (at 231.902 115.824 0)
-    (effects (font (size 1.27 1.27)) (justify left bottom))
-  )
-  (label "B03" (at 231.902 123.444 0)
     (effects (font (size 1.27 1.27)) (justify left bottom))
   )
@@
     (effects (font (size 1.27 1.27)) (justify left bottom))
   )
-  (label "B14" (at 231.902 141.224 0)
+  (label "B0_EN" (at 231.902 123.444 0)
+    (effects (font (size 1.27 1.27)) (justify left bottom))
+  )
+  (label "SCL" (at 257.81 30.734 0)
     (effects (font (size 1.27 1.27)) (justify left bottom))
   )
@@
     (effects (font (size 1.27 1.27)) (justify left bottom))
   )
-  (label "3v2_EN" (at 231.902 108.204 0)
-    (effects (font (size 1.27 1.27)) (justify left bottom))
-  )
-  (label "B04" (at 231.902 128.524 0)
+  (label "B11" (at 231.902 110.744 0)
+    (effects (font (size 1.27 1.27)) (justify left bottom))
+  )
+  (label "B1_EN" (at 231.902 146.304 0)
     (effects (font (size 1.27 1.27)) (justify left bottom))
   )
@@
     (effects (font (size 1.27 1.27)) (justify left bottom))
   )
+  (label "B03" (at 231.902 133.604 0)
+    (effects (font (size 1.27 1.27)) (justify left bottom))
+  )
+  (label "B02" (at 231.902 136.144 0)
+    (effects (font (size 1.27 1.27)) (justify left bottom))
+  )
   (label "B01" (at 121.666 23.368 0)
     (effects (font (size 1.27 1.27)) (justify left bottom))
@@
     (effects (font (size 1.27 1.27)) (justify left bottom))
   )
-  (label "B0_EN" (at 231.902 110.744 0)
-    (effects (font (size 1.27 1.27)) (justify left bottom))
-  )
-  (label "B01" (at 231.902 118.364 0)
+  (label "B04" (at 231.902 131.064 0)
+    (effects (font (size 1.27 1.27)) (justify left bottom))
+  )
+  (label "2v7_EN" (at 231.902 120.904 0)
     (effects (font (size 1.27 1.27)) (justify left bottom))
   )
@@
   )
   (label "VCC1" (at 121.666 49.022 0)
-    (effects (font (size 1.27 1.27)) (justify left bottom))
-  )
-  (label "B02" (at 231.902 120.904 0)
     (effects (font (size 1.27 1.27)) (justify left bottom))
   )
@@
     (effects (font (size 1.27 1.27)) (justify right bottom))
   )
+  (label "B13" (at 231.902 115.824 0)
+    (effects (font (size 1.27 1.27)) (justify left bottom))
+  )
+  (label "B14" (at 231.902 118.364 0)
+    (effects (font (size 1.27 1.27)) (justify left bottom))
+  )
   (label "B12" (at 121.666 82.804 0)
     (effects (font (size 1.27 1.27)) (justify left bottom))
   )
   (label "2v7" (at 218.948 67.31 0)
-    (effects (font (size 1.27 1.27)) (justify left bottom))
-  )
-  (label "B11" (at 231.902 133.604 0)
-    (effects (font (size 1.27 1.27)) (justify left bottom))
-  )
-  (label "SDA" (at 257.81 30.734 0)
     (effects (font (size 1.27 1.27)) (justify left bottom))
   )
@@
     (effects (font (size 1.27 1.27)) (justify left bottom))
   )
-  (label "B1_EN" (at 231.902 113.284 0)
-    (effects (font (size 1.27 1.27)) (justify left bottom))
-  )
   (label "B00" (at 121.666 19.05 0)
     (effects (font (size 1.27 1.27)) (justify left bottom))
@@
     (effects (font (size 1.27 1.27)) (justify left bottom))
   )
-  (label "B10" (at 231.902 131.064 0)
-    (effects (font (size 1.27 1.27)) (justify left bottom))
-  )
   (label "A1" (at 149.86 160.782 0)
+    (effects (font (size 1.27 1.27)) (justify left bottom))
+  )
+  (label "B01" (at 231.902 138.684 0)
     (effects (font (size 1.27 1.27)) (justify left bottom))
   )
@@
     (effects (font (size 1.27 1.27)) (justify left bottom))
   )
+  (label "B12" (at 231.902 113.284 0)
+    (effects (font (size 1.27 1.27)) (justify left bottom))
+  )
   (label "A0" (at 196.342 146.304 180)
     (effects (font (size 1.27 1.27)) (justify right bottom))
+  )
+  (label "B00" (at 231.902 141.224 0)
+    (effects (font (size 1.27 1.27)) (justify left bottom))
+  )
+  (label "3v2_EN" (at 231.902 143.764 0)
+    (effects (font (size 1.27 1.27)) (justify left bottom))
   )
   (symbol (lib_id "power:GND") (at 219.964 42.926 0) (unit 1)
@@
     (pin "9")
   )
+  (symbol (lib_id "power:VCC") (at 214.122 98.044 0) (unit 1)
+    (in_bom yes) (on_board yes)
+    (property "Reference" "#PWR0164" (id 0) (at 214.122 101.854 0)
+      (effects (font (size 1.27 1.27)) hide)
+    )
+    (property "Value" "VCC" (id 1) (at 214.122 91.44 90)
+      (effects (font (size 1.27 1.27)) (justify right))
+    )
+    (property "Footprint" "" (id 2) (at 214.122 98.044 0)
+      (effects (font (size 1.27 1.27)) hide)
+    )
+    (property "Datasheet" "" (id 3) (at 214.122 98.044 0)
+      (effects (font (size 1.27 1.27)) hide)
+    )
+    (pin "1")
+  )
   (symbol (lib_id "power:GND") (at 208.788 44.704 0) (unit 1)
     (in_bom yes) (on_board yes) (fields_autoplaced)
@@
       (reference "#PWR0163") (unit 1) (value "GND") (footprint "")
     )
+    (path "/7b657a65-b914-4b8f-a083-35966e5e5892"
+      (reference "#PWR0164") (unit 1) (value "VCC") (footprint "")
+    )
     (path "/6f984717-b66f-4565-a9e5-0ae595ed9dcc"
