File: EE/Sensing/SensorBoard/Bank0.kicad_sch (KiCad schematic)
At the start: 35 parts

Commit message: WIP - TBs ordered, Sensor board pre layout sensor board
Parts:
- removed D? (x5): LED_Dual_KKA, symbol Device:LED_Dual_KKA
- removed R? (x10): R, Resistor_SMD:R_0402_1005Metric_Pad0.72x0.64mm_HandSolder, symbol Device:R
- added D1, D2, D3, D4, D5: LED_Dual_KKA, Package_TO_SOT_SMD:SC-59, symbol Device:LED_Dual_KKA
- added Q1, Q2, Q3, Q4, Q5: BSS84DW, Package_TO_SOT_SMD:SOT-363_SC-70-6, symbol New_Library:BSS84DW
- added R10, R11, R14, R15, R18, R19, R22, R3, R6, R7: 100k_NP, Resistor_SMD:R_0402_1005Metric_Pad0.72x0.64mm_HandSolder, symbol Device:R
- added R12, R13, R16, R17, R20, R21, R4, R5, R8, R9: 500, Resistor_SMD:R_0402_1005Metric_Pad0.72x0.64mm_HandSolder, symbol Device:R
- J11, J12, J21, J22, J31, J32, J41, J42, J51, J52: renamed from J?; footprint (none) -> Library:TestPattern0
- gave numbers to parts that had none: 10
Connections:
- net GND: now also Q1.1 (S2), Q1.4 (S1), Q2.1 (S2), Q2.4 (S1), Q3.1 (S2), Q3.4 (S1), Q4.1 (S2), Q4.4 (S1), Q5.1 (S2), Q5.4 (S1)
- net H0_0: now also Q1.2 (G2), R3.2
- net H0_1: now also Q2.2 (G2), R7.2
- net H0_2: now also Q3.2 (G2), R11.2
- net H0_3: now also Q4.2 (G2), R15.2
- net H0_4: now also Q5.2 (G2), R19.2
- net H1_0: now also Q1.5 (G1), R6.2
- net H1_1: now also Q2.5 (G1), R10.2
- net H1_2: now also Q3.5 (G1), R14.2
- net H1_3: now also Q4.5 (G1), R18.2
- net H1_4: now also Q5.5 (G1), R22.2
- net VCC: now also D1.3 (A), D2.3 (A), D3.3 (A), D4.3 (A), D5.3 (A), R10.1, R11.1, R14.1, R15.1, R18.1, R19.1, R22.1, R3.1, R6.1, R7.1
- new net: D3.1 (K1), R13.1
- new net: Q3.3 (D1), R13.2
- new net: D2.1 (K1), R9.1
- new net: D2.2 (K2), R8.1
- new net: D1.1 (K1), R5.1
- new net: Q1.3 (D1), R5.2
- new net: Q1.6 (D2), R4.2
- new net: Q3.6 (D2), R12.2
- new net: D1.2 (K2), R4.1
- new net: D4.1 (K1), R17.1
- new net: D4.2 (K2), R16.1
- new net: Q4.3 (D1), R17.2
- new net: Q4.6 (D2), R16.2
- new net: D5.1 (K1), R21.1
- new net: D5.2 (K2), R20.1
- new net: Q5.3 (D1), R21.2
- new net: Q2.3 (D1), R9.2
- new net: Q5.6 (D2), R20.2
- new net: D3.2 (K2), R12.1
- new net: Q2.6 (D2), R8.2
Other:
- moved on the sheet: J11, J12, J21, J22, J31, J32, J41, J42, J51, J52, U11, U12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

Commit message: WIP - Moving Sensor to IO Expander
Connections:
- net VCC: no longer U11.1 (VDD), U21.1 (VDD), U31.1 (VDD), U41.1 (VDD), U51.1 (VDD)
- new net VCC2: U11.1 (VDD), U21.1 (VDD), U31.1 (VDD), U41.1 (VDD), U51.1 (VDD)
Changed lines of the file:
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@@
+    (effects (font (size 1.27 1.27)) (justify left bottom))
+  )
+  (label "VCC2" (at 46.228 29.972 0)
     (effects (font (size 1.27 1.27)) (justify left bottom))
   )
@@
     (effects (font (size 1.27 1.27)) (justify left bottom))
   )
+  (label "VCC2" (at 95.25 31.242 0)
+    (effects (font (size 1.27 1.27)) (justify left bottom))
+  )
   (label "HO_3" (at 198.628 146.558 180)
     (effects (font (size 1.27 1.27)) (justify right bottom))
@@
     (effects (font (size 1.27 1.27)) (justify left bottom))
   )
-  (label "VCC" (at 95.25 31.242 0)
-    (effects (font (size 1.27 1.27)) (justify left bottom))
-  )
   (label "H1_0" (at 277.876 16.764 180)
     (effects (font (size 1.27 1.27)) (justify right bottom))
@@
     (effects (font (size 1.27 1.27)) (justify left bottom))
   )
-  (label "VCC" (at 46.228 29.972 0)
-    (effects (font (size 1.27 1.27)) (justify left bottom))
-  )
   (label "VCC" (at 182.372 137.668 0)
     (effects (font (size 1.27 1.27)) (justify left bottom))
@@
     (effects (font (size 1.27 1.27)) (justify right bottom))
   )
-  (label "VCC" (at 142.24 31.496 0)
-    (effects (font (size 1.27 1.27)) (justify left bottom))
+  (label "VCC2" (at 277.876 43.942 180)
+    (effects (font (size 1.27 1.27)) (justify right bottom))
   )
   (label "VCC" (at 190.246 60.452 0)
     (effects (font (size 1.27 1.27)) (justify left bottom))
   )
+  (label "VCC2" (at 233.172 31.242 0)
+    (effects (font (size 1.27 1.27)) (justify left bottom))
+  )
   (label "VCC" (at 216.916 111.506 0)
     (effects (font (size 1.27 1.27)) (justify left bottom))
@@
     (effects (font (size 1.27 1.27)) (justify left bottom))
   )
+  (label "VCC2" (at 190.246 32.766 0)
+    (effects (font (size 1.27 1.27)) (justify left bottom))
+  )
   (label "HO_1" (at 110.49 155.194 180)
     (effects (font (size 1.27 1.27)) (justify right bottom))
@@
     (effects (font (size 1.27 1.27)) (justify right bottom))
   )
-  (label "VCC" (at 190.246 32.766 0)
-    (effects (font (size 1.27 1.27)) (justify left bottom))
-  )
-  (label "VCC" (at 233.172 31.242 0)
-    (effects (font (size 1.27 1.27)) (justify left bottom))
-  )
   (label "HO_4" (at 240.792 41.402 0)
     (effects (font (size 1.27 1.27)) (justify left bottom))
@@
     (effects (font (size 1.27 1.27)) (justify left bottom))
   )
+  (label "VCC2" (at 142.24 31.496 0)
+    (effects (font (size 1.27 1.27)) (justify left bottom))
+  )
   (label "VCC" (at 203.962 138.938 0)
     (effects (font (size 1.27 1.27)) (justify left bottom))
@@
     (effects (font (size 1.27 1.27)) (justify left))
   )
+  (hierarchical_label "VCC2" (shape input) (at 277.876 43.942 0)
+    (effects (font (size 1.27 1.27)) (justify left))
+  )

Commit message: Fix of Multiplexing
Connections:
- net H1_0 is gone; now on net H0_0: Q1.5 (G1), R6.2, U12.2 (OUTPUT)
- net H1_1 is gone; now on net H0_1: Q2.5 (G1), R10.2, U22.2 (OUTPUT)
- net H1_2 is gone; now on net H0_2: Q3.5 (G1), R14.2, U32.2 (OUTPUT)
- net H1_3 is gone; now on net H0_3: Q4.5 (G1), R18.2, U42.2 (OUTPUT)
- net H1_4 is gone; now on net H0_4: Q5.5 (G1), R22.2, U52.2 (OUTPUT)
- net VCC renamed LED_VCC
- net LED_VCC: no longer U12.1 (VDD), U22.1 (VDD), U32.1 (VDD), U42.1 (VDD), U52.1 (VDD)
- net VCC2 renamed B0_VCC
- new net B1_VCC: U12.1 (VDD), U22.1 (VDD), U32.1 (VDD), U42.1 (VDD), U52.1 (VDD)

Commit message: Replacement after sensing change
Parts:
- removed Q1, Q2, Q3, Q4, Q5: BSS84DW, Package_TO_SOT_SMD:SOT-363_SC-70-6, symbol New_Library:BSS84DW
- removed R10, R11, R14, R15, R18, R19, R22, R3, R6, R7: 100k_NP, Resistor_SMD:R_0402_1005Metric_Pad0.72x0.64mm_HandSolder, symbol Device:R
- D1, D2, D3, D4, D5: footprint Package_TO_SOT_SMD:SC-59 -> Package_TO_SOT_SMD:SOT-23
- U11, U12, U21, U22, U31, U32, U41, U42, U51, U52: value AH1381 -> DRV5032AJDBZR
Connections:
- net H0_0: now also R4.2; no longer U12.2 (OUTPUT)
- net H0_1: now also R8.2; no longer U22.2 (OUTPUT)
- net H0_2: now also R12.2; no longer U32.2 (OUTPUT)
- net H0_3: now also R16.2; no longer U42.2 (OUTPUT)
- net H0_4: now also R20.2; no longer U52.2 (OUTPUT)
- net H1_2: now reaches R13.2
- net H1_2: now also U32.2 (OUTPUT)
- net H1_0: now reaches R5.2
- net H1_0: now also U12.2 (OUTPUT)
- net H1_3: now reaches R17.2
- net H1_3: now also U42.2 (OUTPUT)
- net H1_4: now reaches R21.2
- net H1_4: now also U52.2 (OUTPUT)
- net H1_1: now reaches R9.2
- net H1_1: now also U22.2 (OUTPUT)
