File: EE/Rev2/Main/Motherboard/Power.kicad_sch (KiCad schematic)
At the start: 28 parts, among them J8 Conn_01x02_Male, P1 USB_C_Plug_USB2.0, Q1 Q_PMOS_GSD, Q2 Q_NMOS_GSD, SW1 SW_DPST, U2 MCP73832-2-OT, U5 LM3670MF-3.3

Commit message: Updating Format, Adding Rev2 Start
Connections:
- net VBAT_ADC: no longer U5.3 (EN)
Other:
- note added: "TODO this is a brown out circuit. Not a real power down circuit. Do more modelling on physical devices first"
- moved on the sheet: C2, C4, C6, C8, D1, J8, L2, P1, Q1, Q2, R10, R11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
